File: kicad/seven_segment_display/seven_segment_display.kicad_sch (KiCad schematic)
At the start: 11 parts, among them J3 Conn_01x12_Pin, U1 74AHC595

Commit message: final pcb design completed
Connections:
- net CLK: now also J3.5 (Pin_5); no longer J3.8 (Pin_8)
- net LATCH: now also J3.6 (Pin_6); no longer J3.7 (Pin_7)
- net SER: now also J3.8 (Pin_8); no longer J3.5 (Pin_5)
- net ~OE: now also J3.7 (Pin_7); no longer J3.6 (Pin_6)
Changed lines of the file:
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@@
+		)
+	)
+	(label "SER"
+		(at 76.2 77.47 0)
+		(effects
+			(font
+				(size 1.27 1.27)
+			)
+			(justify left bottom)
 		)
 	)
@@
 	)
 	(label "~OE"
-		(at 76.2 72.39 0)
-		(effects
-			(font
-				(size 1.27 1.27)
-			)
-			(justify left bottom)
-		)
-	)
-	(label "SER"
-		(at 76.2 69.85 0)
+		(at 76.2 74.93 0)
 		(effects
 			(font
@@
 		)
 	)
+	(label "CLK"
+		(at 76.2 69.85 0)
+		(effects
+			(font
+				(size 1.27 1.27)
+			)
+			(justify left bottom)
+		)
+	)
 	(label "DIG3"
 		(at 220.98 95.25 0)
@@
 	)
 	(label "LATCH"
-		(at 76.2 74.93 0)
+		(at 76.2 72.39 0)
 		(effects
 			(font
@@
 		(effects
 			(font
-				(size 1.27 1.27)
-			)
-			(justify left bottom)
-		)
-	)
-	(label "CLK"
-		(at 76.2 77.47 0)
-		(effects
-			(font
